File: MiniTune v1.0/MiniTune v0.1.kicad_sch (KiCad schematic)
At the start: 13 parts

Commit message: Added schematics
Parts:
- added C? (x2): 47uF, Capacitor_SMD:C_0805_2012Metric_Pad1.18x1.45mm_HandSolder, symbol Device:C_Polarized_US
- added FB? (x2): 742792664, Capacitor_SMD:C_0603_1608Metric_Pad1.08x0.95mm_HandSolder, symbol Device:FerriteBead
- added J?: IDC_2x05, Connector_IDC:IDC-Header_2x05_P2.54mm_Vertical, symbol Connector:Conn_01x10_Male
Connections:
- net +12V: now also C?.1, FB?.2
- net -12V: now also C?.2, FB?.2
- net GND: now also C?.1, C?.2, J?.3 (Pin_3), J?.4 (Pin_4), J?.5 (Pin_5), J?.6 (Pin_6), J?.7 (Pin_7), J?.8 (Pin_8)
- new net: FB?.1, J?.1 (Pin_1), J?.2 (Pin_2)
- new net: FB?.1, J?.10 (Pin_10), J?.9 (Pin_9)
Other:
- removed sheet Power
- company: (none) -> benjiaomodular
- title: (none) -> MiniTune
- moved on the sheet: A?, D?, J?, R?, SW_MUTE, U?, U?A, U?B, U?C
